Commit message: Changes to be committed: brainco_hand 	new file:   src/k100_description/meshes/k100/brainco_left_wrist_yaw_link.STL 	new file:   src/k100_description/meshes/k100/brainco_right_wrist_yaw_link.STL 	modified:   src/k100_description/urdf/k100_brainco.urdf

File: src/k100_description/urdf/k100_brainco.urdf (robot description, URDF)
Before this commit: robot k100, 60 links, 59 joints
Links:
- link left_wrist_yaw_link: geometry collision mesh filename=package://k100_description/meshes/k100/brainco_left_wrist_y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; visual mesh filename=package://k100_description/meshes/k100/brainco_left_wrist_y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
- link right_wrist_yaw_link: geometry collision mesh filename=package://k100_description/meshes/k100/brainco_ right_wrist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; visual mesh filename=package://k100_description/meshes/k100/brainco_right_wrist_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
Joints:
- joint L_base_link_joint: origin xyz=-0.0268 0.005 -0.051 rpy=3.14159 0 -1.5708 -> xyz=-0.0268 0.000 -0.081 rpy=3.14159 0 -1.5708
- joint R_base_link_joint: origin xyz=-0.0268 -0.005 -0.051 rpy=3.14159 0 1.5708 -> xyz=-0.0268 0.000 -0.081 rpy=3.14159 0 1.5708

Commit message: Changes to be committed: 兼容泰科控制器旋转方向和初始角度 	modified:   src/k100_brainco_moveit_config/config/initial_positions.yaml 	modified:   src/k100_description/urdf/k100_brainco.urdf

File: src/k100_description/urdf/k100_brainco.urdf (robot description, URDF)
Before this commit: robot k100, 60 links, 59 joints
Joints:
- joint left_elbow_joint: limit lower=-1.5707963267948966 upper=2.871066619530672 effort=10 velocity=100 -> lower=-0.260 upper=2.355 effort=10 velocity=100
- joint left_shoulder_pitch_joint: axis 0 0 1 -> 0 0 -1; limit lower=-3.0229102644541785 upper=3.005456971934235 effort=10 velocity=100 -> lower=-2.966 upper=2.966 effort=10 velocity=100
- joint left_shoulder_roll_joint: limit lower=-3.4033920413889422 upper=0.3490658503988659 effort=10 velocity=100 -> lower=-1.047 upper=1.5708 effort=10 velocity=100; origin xyz=-0.052528 0 0.057497 rpy=1.5708 0 0 -> xyz=-0.052528 0 0.057497 rpy=-3.14159 0 0
- joint left_shoulder_yaw_joint: limit lower=-1.5707963267948966 upper=3.141592653589793 effort=10 velocity=100 -> lower=-2.966 upper=2.966 effort=10 velocity=100; origin xyz=0.052528 0 -0.1236 rpy=0 0 0 -> xyz=0.052528 0 -0.1236 rpy=0 0 -1.5708
- joint left_wrist_pitch_joint: limit lower=-1.8151424220741028 upper=1.8849555921538759 effort=10 velocity=100 -> lower=-2.966 upper=-0.262 effort=10 velocity=100; origin xyz=0.0017429 -0.03829 -0.152 rpy=0 0 0 -> xyz=0.0017429 -0.03829 -0.152 rpy=0 -1.5708 0
- joint left_wrist_roll_joint: limit lower=-2.9670597283903604 upper=3.01941960595019 effort=10 velocity=100 -> lower=-2.966 upper=2.966 effort=10 velocity=100
- joint left_wrist_yaw_joint: limit lower=-1.5707963267948966 upper=1.605702911834783 effort=10 velocity=100 -> lower=-1.31 upper=1.22 effort=10 velocity=100
- joint right_elbow_joint: limit lower=-1.5533430342749535 upper=2.897246558310587 effort=10 velocity=100 -> lower=-0.260 upper=2.355 effort=10 velocity=100
- joint right_shoulder_pitch_joint: axis 0 0 -1 -> 0 0 1; limit lower=-3.0229102644541785 upper=3.005456971934235 effort=10 velocity=100 -> lower=-2.966 upper=2.966 effort=10 velocity=100
- joint right_shoulder_roll_joint: limit lower=-3.4033920413889422 upper=0.29670597283903605 effort=10 velocity=100 -> lower=-1.047 upper=1.5708 effort=10 velocity=100; origin xyz=0 0 0.063497 rpy=-1.5708 0 0 -> xyz=0 0 0.063497 rpy=-3.14159 0 0
- joint right_shoulder_yaw_joint: axis 0 0 1 -> 0 0 -1; limit lower=-1.5707963267948966 upper=3.141592653589793 effort=10 velocity=100 -> lower=-2.966 upper=2.966 effort=10 velocity=100; origin xyz=0 0 -0.1236 rpy=0 0 0 -> xyz=0 0 -0.1236 rpy=0 0 1.5708
- joint right_wrist_pitch_joint: limit lower=-1.8325957145940461 upper=1.8325957145940461 effort=10 velocity=100 -> lower=-2.966 upper=-0.262 effort=10 velocity=100; origin xyz=0.0017429 -0.03829 -0.152 rpy=0 0 0 -> xyz=0.0017429 -0.03829 -0.152 rpy=0 -1.5708 0
- joint right_wrist_roll_joint: axis 0 0 1 -> 0 0 -1; limit lower=-1.8325957145940461 upper=1.8325957145940461 effort=10 velocity=100 -> lower=-2.966 upper=2.966 effort=10 velocity=100
- joint right_wrist_yaw_joint: axis -1 0 0 -> 1 0 0; limit lower=-1.5882496193148399 upper=1.5882496193148399 effort=10 velocity=100 -> lower=-1.31 upper=1.22 effort=10 velocity=100
