Commit message: Changes to be committed:add both_arms group,fix some bugs

File: src/k100_brainco_moveit_config/config/k100.ros2_control.xacro (robot description, xacro)
@@ -120,4 +120,46 @@
                 <state_interface name="velocity"/>
             </joint>
+            <joint name="left_index_proximal_joint">
+                <command_interface name="position"/>
+                <state_interface name="position">
+                  <param name="initial_value">${initial_positions['left_index_proximal_joint']}</param>
+                </state_interface>
+                <state_interface name="velocity"/>
+            </joint>
+            <joint name="left_middle_proximal_joint">
+                <command_interface name="position"/>
+                <state_interface name="position">
+                  <param name="initial_value">${initial_positions['left_middle_proximal_joint']}</param>
+                </state_interface>
+                <state_interface name="velocity"/>
+            </joint>
+            <joint name="left_pinky_proximal_joint">
+                <command_interface name="position"/>
+                <state_interface name="position">
+                  <param name="initial_value">${initial_positions['left_pinky_proximal_joint']}</param>
+                </state_interface>
+                <state_interface name="velocity"/>
+            </joint>
+            <joint name="left_ring_proximal_joint">
+                <command_interface name="position"/>
+                <state_interface name="position">
+                  <param name="initial_value">${initial_positions['left_ring_proximal_joint']}</param>
+                </state_interface>
+                <state_interface name="velocity"/>
+            </joint>
+            <joint name="left_thumb_metacarpal_joint">
+                <command_interface name="position"/>
+                <state_interface name="position">
+                  <param name="initial_value">${initial_positions['left_thumb_metacarpal_joint']}</param>
+                </state_interface>
+                <state_interface name="velocity"/>
+            </joint>
+            <joint name="left_thumb_proximal_joint">
+                <command_interface name="position"/>
+                <state_interface name="position">
+                  <param name="initial_value">${initial_positions['left_thumb_proximal_joint']}</param>
+                </state_interface>
+                <state_interface name="velocity"/>
+            </joint>
             <joint name="right_index_proximal_joint">
                 <command_interface name="position"/>
@@ -127,11 +169,4 @@
                 <state_interface name="velocity"/>
             </joint>
-            <joint name="right_index_tip_joint">
-                <command_interface name="position"/>
-                <state_interface name="position">
-                  <param name="initial_value">${initial_positions['right_index_tip_joint']}</param>
-                </state_interface>
-                <state_interface name="velocity"/>
-            </joint>
             <joint name="right_middle_proximal_joint">
                 <command_interface name="position"/>
@@ -141,11 +176,4 @@
                 <state_interface name="velocity"/>
             </joint>
-            <joint name="right_middle_tip_joint">
-                <command_interface name="position"/>
-                <state_interface name="position">
-                  <param name="initial_value">${initial_positions['right_middle_tip_joint']}</param>
-                </state_interface>
-                <state_interface name="velocity"/>
-            </joint>
             <joint name="right_pinky_proximal_joint">
                 <command_interface name="position"/>
@@ -155,11 +183,4 @@
                 <state_interface name="velocity"/>
             </joint>
-            <joint name="right_pinky_tip_joint">
-                <command_interface name="position"/>
-                <state_interface name="position">
-                  <param name="initial_value">${initial_positions['right_pinky_tip_joint']}</param>
-                </state_interface>
-                <state_interface name="velocity"/>
-            </joint>
             <joint name="right_ring_proximal_joint">
                 <command_interface name="position"/>
@@ -169,11 +190,4 @@
                 <state_interface name="velocity"/>
             </joint>
-            <joint name="right_ring_tip_joint">
-                <command_interface name="position"/>
-                <state_interface name="position">
-                  <param name="initial_value">${initial_positions['right_ring_tip_joint']}</param>
-                </state_interface>
-                <state_interface name="velocity"/>
-            </joint>
             <joint name="right_thumb_metacarpal_joint">
                 <command_interface name="position"/>
@@ -187,88 +201,4 @@
                 <state_interface name="position">
                   <param name="initial_value">${initial_positions['right_thumb_proximal_joint']}</param>
-                </state_interface>
-                <state_interface name="velocity"/>
-            </joint>
-            <joint name="right_thumb_tip">
-                <command_interface name="position"/>
-                <state_interface name="position">
-                  <param name="initial_value">${initial_positions['right_thumb_tip']}</param>
-                </state_interface>
-                <state_interface name="velocity"/>
-            </joint>
-            <joint name="left_index_proximal_joint">
-                <command_interface name="position"/>
-                <state_interface name="position">
-                  <param name="initial_value">${initial_positions['left_index_proximal_joint']}</param>
-                </state_interface>
-                <state_interface name="velocity"/>
-            </joint>
-            <joint name="left_index_tip_joint">
-                <command_interface name="position"/>
-                <state_interface name="position">
-                  <param name="initial_value">${initial_positions['left_index_tip_joint']}</param>
-                </state_interface>
-                <state_interface name="velocity"/>
-            </joint>
-            <joint name="left_middle_proximal_joint">
-                <command_interface name="position"/>
-                <state_interface name="position">
-                  <param name="initial_value">${initial_positions['left_middle_proximal_joint']}</param>
-                </state_interface>
-                <state_interface name="velocity"/>
-            </joint>
-            <joint name="left_middle_tip_joint">
-                <command_interface name="position"/>
-                <state_interface name="position">
-                  <param name="initial_value">${initial_positions['left_middle_tip_joint']}</param>
-                </state_interface>
-                <state_interface name="velocity"/>
-            </joint>
-            <joint name="left_pinky_proximal_joint">
-                <command_interface name="position"/>
-                <state_interface name="position">
-                  <param name="initial_value">${initial_positions['left_pinky_proximal_joint']}</param>
-                </state_interface>
-                <state_interface name="velocity"/>
-            </joint>
-            <joint name="left_pinky_tip_joint">
-                <command_interface name="position"/>
-                <state_interface name="position">
-                  <param name="initial_value">${initial_positions['left_pinky_tip_joint']}</param>
-                </state_interface>
-                <state_interface name="velocity"/>
-            </joint>
-            <joint name="left_ring_proximal_joint">
-                <command_interface name="position"/>
-                <state_interface name="position">
-                  <param name="initial_value">${initial_positions['left_ring_proximal_joint']}</param>
-                </state_interface>
-                <state_interface name="velocity"/>
-            </joint>
-            <joint name="left_ring_tip_joint">
-                <command_interface name="position"/>
-                <state_interface name="position">
-                  <param name="initial_value">${initial_positions['left_ring_tip_joint']}</param>
-                </state_interface>
-                <state_interface name="velocity"/>
-            </joint>
-            <joint name="left_thumb_metacarpal_joint">
-                <command_interface name="position"/>
-                <state_interface name="position">
-                  <param name="initial_value">${initial_positions['left_thumb_metacarpal_joint']}</param>
-                </state_interface>
-                <state_interface name="velocity"/>
-            </joint>
-            <joint name="left_thumb_proximal_joint">
-                <command_interface name="position"/>
-                <state_interface name="position">
-                  <param name="initial_value">${initial_positions['left_thumb_proximal_joint']}</param>
-                </state_interface>
-                <state_interface name="velocity"/>
-            </joint>
-            <joint name="left_thumb_tip_joint">
-                <command_interface name="position"/>
-                <state_interface name="position">
-                  <param name="initial_value">${initial_positions['left_thumb_tip_joint']}</param>
                 </state_interface>
                 <state_interface name="velocity"/>

File: src/k100_description/urdf/k100_braincowithcolor.urdf (robot description, URDF)
Before this commit: robot k100, 64 links, 63 joints
Links:
- removed link left_arm_base_link
- removed link left_arm_ee_link
- removed link left_hand_base_link
- removed link right_arm_base_link
- removed link right_arm_ee_link
- removed link right_hand_base_link
- added link left_base_link, mass 0.238; collision mesh filename=package://k100_description/meshes/meshes_brainco/left_base_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; visual mesh filename=package://k100_description/meshes/meshes_brainco/left_base_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
- added link right_base_link, mass 0.238; collision mesh filename=package://k100_description/meshes/meshes_brainco/right_base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; visual mesh filename=package://k100_description/meshes/meshes_brainco/right_base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
- link base_link: geometry collision mesh filename=package://k100_description/meshes/k100/base_link.dae; visual mesh filename=package://k100_description/meshes/k100/base_link.dae
- link head_pitch_link: geometry collision mesh filename=package://k100_description/meshes/k100/head_pitch_link.dae; visual mesh filename=package://k100_description/meshes/k100/head_pitch_link.dae
- link head_yaw_link: geometry collision mesh filename=package://k100_description/meshes/k100/head_yaw_link.dae; visual mesh filename=package://k100_description/meshes/k100/head_yaw_link.dae
- link left_elbow_link: geometry collision mesh filename=package://k100_description/meshes/k100/left_elbow_link.dae; visual mesh filename=package://k100_description/meshes/k100/left_elbow_link.dae
- link right_elbow_link: geometry collision mesh filename=package://k100_description/meshes/k100/right_elbow_link.dae; visual mesh filename=package://k100_description/meshes/k100/right_elbow_link.dae
Joints:
- removed joint left_arm_base_joint
- removed joint left_arm_ee_joint
- removed joint left_hand_base_link_joint
- removed joint right_arm_base_joint
- removed joint right_arm_ee_joint
- removed joint right_hand_base_link_joint
- removed joint right_thumb_tip_joint
- added joint L_base_link_joint: type fixed, parent left_wrist_yaw_link, child left_base_link, origin xyz=-0.0268 0.000 -0.081 rpy=3.14159 0 -1.5708
- added joint R_base_link_joint: type fixed, parent right_wrist_yaw_link, child right_base_link, origin xyz=-0.0268 0.000 -0.081 rpy=3.14159 0 1.5708
- added joint right_thumb_tip: type revolute, parent right_thumb_distal_link, child right_thumb_tip, origin xyz=0 0.026529 -0.0017734 rpy=-0.06675 0 0, axis 1 0 0, limit lower=0 upper=0 effort=0 velocity=0
- joint left_elbow_joint: limit lower=-0.260 upper=2.355 effort=10.0 velocity=100.0 -> lower=-0.260 upper=2.355 effort=10 velocity=100
- joint left_index_proximal_joint: parent left_hand_base_link -> left_base_link
- joint left_index_tip_joint: type fixed -> revolute
- joint left_middle_proximal_joint: parent left_hand_base_link -> left_base_link
- joint left_middle_tip_joint: type fixed -> revolute
- joint left_pinky_proximal_joint: parent left_hand_base_link -> left_base_link
- joint left_pinky_tip_joint: type fixed -> revolute
- joint left_ring_proximal_joint: parent left_hand_base_link -> left_base_link
- joint left_ring_tip_joint: type fixed -> revolute
- joint left_shoulder_pitch_joint: limit lower=-2.966 upper=2.966 effort=10.0 velocity=100.0 -> lower=-2.966 upper=2.966 effort=10 velocity=100; origin xyz=0.0 0.0 0.0121 rpy=0 0 -1.5708 -> xyz=-0.29331 0.15637 1.1789 rpy=-1.5708 0 0; parent left_arm_base_link -> base_link
- joint left_shoulder_roll_joint: limit lower=-1.047 upper=1.5708 effort=10.0 velocity=100.0 -> lower=-1.047 upper=1.5708 effort=10 velocity=100
- joint left_shoulder_yaw_joint: limit lower=-2.966 upper=2.966 effort=10.0 velocity=100.0 -> lower=-2.966 upper=2.966 effort=10 velocity=100
- joint left_thumb_metacarpal_joint: parent left_hand_base_link -> left_base_link
- joint left_thumb_tip_joint: type fixed -> revolute
- joint left_wrist_pitch_joint: limit lower=-2.966 upper=-0.262 effort=10.0 velocity=100.0 -> lower=-2.966 upper=-0.262 effort=10 velocity=100
- joint left_wrist_roll_joint: limit lower=-2.966 upper=2.966 effort=10.0 velocity=100.0 -> lower=-2.966 upper=2.966 effort=10 velocity=100
- joint left_wrist_yaw_joint: limit lower=-1.31 upper=1.22 effort=10.0 velocity=100.0 -> lower=-1.31 upper=1.22 effort=10 velocity=100
- joint right_elbow_joint: limit lower=-0.260 upper=2.355 effort=10.0 velocity=100.0 -> lower=-0.260 upper=2.355 effort=10 velocity=100
- joint right_index_proximal_joint: parent right_hand_base_link -> right_base_link
- joint right_index_tip_joint: type fixed -> revolute
- joint right_middle_proximal_joint: parent right_hand_base_link -> right_base_link
- joint right_middle_tip_joint: type fixed -> revolute
- joint right_pinky_proximal_joint: parent right_hand_base_link -> right_base_link
- joint right_pinky_tip_joint: type fixed -> revolute
- joint right_ring_proximal_joint: parent right_hand_base_link -> right_base_link
- joint right_ring_tip_joint: type fixed -> revolute
- joint right_shoulder_pitch_joint: limit lower=-2.966 upper=2.966 effort=10.0 velocity=100.0 -> lower=-2.966 upper=2.966 effort=10 velocity=100; origin xyz=0.0 0.0 0.0121 rpy=0 0 1.5708 -> xyz=-0.29331 -0.15184 1.1789 rpy=1.5708 0 0; parent right_arm_base_link -> base_link
- joint right_shoulder_roll_joint: limit lower=-1.047 upper=1.5708 effort=10.0 velocity=100.0 -> lower=-1.047 upper=1.5708 effort=10 velocity=100
- joint right_shoulder_yaw_joint: limit lower=-2.966 upper=2.966 effort=10.0 velocity=100.0 -> lower=-2.966 upper=2.966 effort=10 velocity=100
- joint right_thumb_metacarpal_joint: parent right_hand_base_link -> right_base_link
- joint right_wrist_pitch_joint: limit lower=-2.966 upper=-0.262 effort=10.0 velocity=100.0 -> lower=-2.966 upper=-0.262 effort=10 velocity=100
- joint right_wrist_roll_joint: limit lower=-2.966 upper=2.966 effort=10.0 velocity=100.0 -> lower=-2.966 upper=2.966 effort=10 velocity=100
- joint right_wrist_yaw_joint: limit lower=-1.31 upper=1.22 effort=10.0 velocity=100.0 -> lower=-1.31 upper=1.22 effort=10 velocity=100
